Commit message: rviz urdf update

File: platform_description/xacro/urdf/wam_platform.urdf (robot description, URDF)
Before this commit: robot wam, 19 links, 18 joints
Links:
- added link segment_top, mass 500.0; collision cylinder length=0.4 radius=0.02; visual cylinder length=0.4 radius=0.02
- link p0_link: geometry collision cylinder length=0.05 radius=0.1; visual cylinder length=0.05 radius=0.1
Joints:
- added joint top_joint: type fixed, parent segment_top, child platform_top_link, origin xyz=0.4 0 0 rpy=0 0 0
- joint imu_joint: origin xyz=0.0 -0.24 0.0525 rpy=0 0 0 -> xyz=0.0525 0 -0.16 rpy=1.57079632679 0 1.57079632679
- joint p0_joint: origin xyz=0 0.275 0 rpy=1.57079632679 0 1.57079632679 -> xyz=0 0.05 0 rpy=1.57079632679 0 1.57079632679
- joint p1_joint: child platform_top_link -> segment_top
