Commit message: added GazeboRosImuSensor

File: platform_description/xacro/platform.urdf.xacro (robot description, xacro)
@@ -94,5 +94,5 @@
            </actuator>
   </transmission>
- <!-- platformtop height is .55+.01+.025=.585 -->
+ <!-- platformtop -->
   <link name="platform_top_link">
     <inertial>
@@ -146,4 +146,52 @@
            </actuator>
   </transmission>
+  <!-- IMU -->
+  <link name="imu_link">
+    <inertial>
+      <mass value="0.001"/>
+      <origin rpy="0.0 0.0 0.0" xyz="0 0 0"/>
+      <inertia ixx="0.0001" ixy="0" ixz="0" iyy="0.000001" iyz="0" izz="0.0001"/>
+    </inertial>
+    <visual>
+      <origin rpy="0 0 0" xyz="0 0 0"/>
+      <geometry>
+        <box size="0.01 0.01 0.01"/>
+      </geometry>
+    </visual>
+    <collision>
+      <origin rpy="0 0 0" xyz="0 0 0"/>
+      <geometry>
+        <box size=".001 .001 .001"/>
+      </geometry>
+    </collision>
+  </link>
+  <gazebo reference="imu_link">
+    <material>Gazebo/Green</material>
+  </gazebo>
+  <!-- IMU joint -->
+  <joint name="imu_joint" type="fixed">
+    <axis xyz="1 0 0"/> <!-- 0 1 0 -->
+    <origin xyz="0 0 0.0"/>
+    <parent link="platform_top_link"/>
+    <child link="imu_link"/>
+  </joint>
+  <!-- The imu sensor -->
+  <gazebo reference="imu_link">
+    <gravity>true</gravity>
+    <sensor name="imu_sensor" type="imu">
+      <always_on>true</always_on>
+      <visualize>true</visualize>
+      <plugin filename="libgazebo_ros_imu_sensor.so" name="imu_plugin">
+        <topicName>/imu/data</topicName>
+        <bodyName>imu_link</bodyName>
+        <updateRateHZ>1000.0</updateRateHZ>
+        <gaussianNoise>0.0</gaussianNoise>
+        <xyzOffset>0 0 0</xyzOffset>
+        <rpyOffset>0 0 0</rpyOffset>
+        <frameName>imu_link</frameName>
+      </plugin>
+      <pose>0 0 0 0 0 0</pose>
+    </sensor>
+  </gazebo>
   <gazebo>
     <!--static>true</static-->

Commit message: gazebo default
mu1, mu2, Kp and Kd

File: platform_description/xacro/platform.urdf.xacro (robot description, xacro)
@@ -36,8 +36,4 @@
   <gazebo reference="p0_link">
     <material>Gazebo/Yellow</material>
-    <mu1>1000.0</mu1>
-    <mu2>1000.0</mu2>
-    <kp>10000000.0</kp>
-    <kd>1.0</kd>
     <selfCollide>true</selfCollide>
   </gazebo>
@@ -51,26 +47,7 @@
                izz="20000000" />
     </inertial>
-    <!-- visual>
-      <origin xyz="0.0 0.0 0.0" rpy="0 0 0" />
-      <geometry>
-        <cylinder radius="${leg_radius}" length="0.0" />
-      </geometry>
-      <material name="Black">
-		<color rgba="0 0 0 1.0"/>
-      </material>
-    </visual>
-    <collision>
-      <origin xyz="0.0 0.0 0.0" rpy="0.0 0.0 0.0" />
-      <geometry>
-        <cylinder radius="${leg_radius}" length="0.0" />
-      </geometry>
-    </collision>-->
   </link>
   <gazebo reference="p1_link">
     <material>Gazebo/Green</material>
-    <mu1>1000.0</mu1>
-    <mu2>1000.0</mu2>
-    <kp>10000000.0</kp>
-    <kd>1.0</kd>
     <selfCollide>true</selfCollide>
   </gazebo>
@@ -121,8 +98,4 @@
   <gazebo reference="platform_top_link">
     <material>Gazebo/Red</material>
-    <mu1>50.0</mu1>
-    <mu2>50.0</mu2>
-    <kp>1000000.0</kp>
-    <kd>1.0</kd>
     <selfCollide>true</selfCollide>
   </gazebo>

File: platform_description/xacro/urdf/platform.urdf (robot description, URDF)
Before this commit: robot platform, 4 links, 3 joints
Links:
- link p1_link: geometry collision cylinder length=0.0 radius=${leg_radius}; visual cylinder length=0.0 radius=${leg_radius}

Commit message: properties urdf
platform geometrical properties in separate file

File: platform_description/xacro/platform.urdf.xacro (robot description, xacro)
@@ -1,20 +1,12 @@
 <?xml version="1.0"?>
 <robot name="platform" xmlns:xacro="http://www.ros.org/wiki/xacro" >
-  <xacro:property name="platform_height" value="0.55" />
-  <xacro:property name="platform_radius" value="0.3" />
-  <xacro:property name="leg_radius" value="0.02" />
-  <xacro:property name="platform_x" value="0.98" />
-  <xacro:property name="platform_y" value="0.0" />
-  <xacro:property name="platform_z" value="0.0" />
-  <xacro:property name="platform_top_thickness" value="0.05"/>
-  <xacro:property name="M_PI" value="3.1415926535897931" />
   <!-- P0 -->
   <link name="p0_link">
     <inertial>
-      <mass value="100.0" />
+      <mass value="800.0" />
       <origin xyz="0.0 0.0 ${platform_height/4}" />
-      <inertia ixx="640208333.333333" ixy="0"  ixz="0"
-               iyy="640208333.333333" iyz="0"
-               izz="20000000" />
+      <inertia ixx="6.4021" ixy="0"  ixz="0"
+               iyy="6.4021" iyz="0"
+               izz="0.2" />
     </inertial>
     <visual>
@@ -71,5 +63,5 @@
            </actuator>
   </transmission>
- <!-- platformtop -->
+ <!-- platform top -->
   <link name="platform_top_link">
     <inertial>
@@ -126,12 +118,12 @@
   <link name="imu_link">
     <inertial>
-      <mass value="0.001"/>
+      <mass value="0.01"/>
       <origin rpy="0.0 0.0 0.0" xyz="0 0 0"/>
-      <inertia ixx="0.0001" ixy="0" ixz="0" iyy="0.000001" iyz="0" izz="0.0001"/>
+      <inertia ixx="0.0077083" ixy="0" ixz="0" iyy="0.0077083" iyz="0" izz="0.0077083"/>
     </inertial>
     <visual>
       <origin rpy="0 0 0" xyz="0 0 0"/>
       <geometry>
-        <box size="0.01 0.01 0.01"/>
+        <box size="0.03 0.03 0.005"/>
       </geometry>
     </visual>

File: platform_description/xacro/wam_platform.urdf.xacro (robot description, xacro)
@@ -1,13 +1,6 @@
 <?xml version="1.0"?>
 <robot name ="wam" xmlns:xacro="http://www.ros.org/wiki/xacro">
-        <xacro:property name="platform_height" value="0.55" />
-        <xacro:property name="platform_radius" value="0.3" />
-        <xacro:property name="leg_radius" value="0.02" />
-        <xacro:property name="platform_x" value="0.98" />
-        <xacro:property name="platform_y" value="0.0" />
-        <xacro:property name="platform_z" value="0.0" />
-        <xacro:property name="platform_top_thickness" value="0.05"/>
-	<xacro:property name="M_PI" value="3.1415926535897931" />
 	<link name="world" />
+	<xacro:include filename="$(find platform_description)/xacro/properties.urdf.xacro" />
 	<xacro:include filename="$(find platform_description)/xacro/platform.urdf.xacro" />
 	<joint name="world_platform_joint" type="fixed">

Commit message: imu inercia

File: platform_description/xacro/platform.urdf.xacro (robot description, xacro)
@@ -4,9 +4,9 @@
   <link name="p0_link">
     <inertial>
-      <mass value="800.0" />
+      <mass value="500.0" />
       <origin xyz="0.0 0.0 ${platform_height/4}" />
-      <inertia ixx="6.4021" ixy="0"  ixz="0"
-               iyy="6.4021" iyz="0"
-               izz="0.2" />
+      <inertia ixx="3.2010" ixy="0"  ixz="0"
+               iyy="3.2010" iyz="0"
+               izz="0.1" />
     </inertial>
     <visual>
@@ -28,4 +28,8 @@
   <gazebo reference="p0_link">
     <material>Gazebo/Yellow</material>
+    <mu1>1000.0</mu1>
+    <mu2>1000.0</mu2>
+    <kp>10000000.0</kp>
+    <kd>1.0</kd>
     <selfCollide>true</selfCollide>
   </gazebo>
@@ -33,13 +37,17 @@
   <link name="p1_link">
     <inertial>
-      <mass value="100.0" />
-      <origin xyz="0.0 0.0 0.0" />
-      <inertia ixx="640208333.333333" ixy="0"  ixz="0"
-               iyy="640208333.333333" iyz="0"
-               izz="20000000" />
+      <mass value="500.0" />
+      <origin xyz="0.1 0.0 0.0" />
+      <inertia ixx="3.2010" ixy="0"  ixz="0"
+               iyy="3.2010" iyz="0"
+               izz="0.1" />
     </inertial>
   </link>
   <gazebo reference="p1_link">
     <material>Gazebo/Green</material>
+    <mu1>1000.0</mu1>
+    <mu2>1000.0</mu2>
+    <kp>10000000.0</kp>
+    <kd>1.0</kd>
     <selfCollide>true</selfCollide>
   </gazebo>
@@ -49,5 +57,5 @@
     <origin xyz="0.0 0.0 ${platform_z+platform_height/2}" rpy="0 0 0" />
     <child link="p1_link" />
-    <limit effort="1000.0" lower="-2.0" upper="2.0" velocity="1.5" />
+    <limit effort="100000.0" lower="-2.0" upper="2.0" velocity="1.5" />
     <axis xyz="0 1 0"/>
   </joint>
@@ -66,9 +74,9 @@
   <link name="platform_top_link">
     <inertial>
-      <mass value="1.0" />
+      <mass value="5.0" />
       <origin xyz="0.0 0.0 ${platform_top_thickness/2}" />
-      <inertia ixx="1" ixy="0"  ixz="0"
-               iyy="1" iyz="0"
-               izz="1" />
+      <inertia ixx="1.0" ixy="0"  ixz="0"
+               iyy="1.0" iyz="0"
+               izz="1.0" />
     </inertial>
     <visual>
@@ -101,5 +109,5 @@
     <origin xyz="0.0 0.0 0.0" rpy="0 0 0" />
     <child link="platform_top_link" />
-    <limit effort="1000.0" lower="-2.0" upper="2.0" velocity="1.5" />
+    <limit effort="100000.0" lower="-2.0" upper="2.0" velocity="1.5" />
     <axis xyz="1 0 0"/>
   </joint>
@@ -120,5 +128,7 @@
       <mass value="0.01"/>
       <origin rpy="0.0 0.0 0.0" xyz="0 0 0"/>
-      <inertia ixx="0.0077083" ixy="0" ixz="0" iyy="0.0077083" iyz="0" izz="0.0077083"/>
+      <inertia ixx="0.00000077083" ixy="0" ixz="0"
+               iyy="0.00000077083" iyz="0"
+               izz="0.00000077083"/>
     </inertial>
     <visual>
@@ -141,5 +151,5 @@
   <joint name="imu_joint" type="fixed">
     <axis xyz="1 0 0"/> <!-- 0 1 0 -->
-    <origin xyz="0 0 0.0"/>
+    <origin rpy="0 0 0" xyz="0 0 0"/>
     <parent link="platform_top_link"/>
     <child link="imu_link"/>

Commit message: imu collision update

File: platform_description/xacro/platform.urdf.xacro (robot description, xacro)
@@ -141,5 +141,5 @@
       <origin rpy="0 0 0" xyz="0 0 0"/>
       <geometry>
-        <box size=".001 .001 .001"/>
+        <box size="0.03 0.03 0.005"/>
       </geometry>
     </collision>

Commit message: wam position to properties
+ imu position changed

File: platform_description/xacro/platform.urdf.xacro (robot description, xacro)
@@ -151,5 +151,5 @@
   <joint name="imu_joint" type="fixed">
     <axis xyz="1 0 0"/> <!-- 0 1 0 -->
-    <origin rpy="0 0 0" xyz="0 0 0"/>
+    <origin rpy="0 0 0" xyz="${wam_x+0.015} ${wam_y-0.02} ${platform_top_thickness+0.0025}"/>
     <parent link="platform_top_link"/>
     <child link="imu_link"/>

File: platform_description/xacro/properties.urdf.xacro (robot description, xacro)
@@ -4,8 +4,12 @@
   <xacro:property name="platform_radius" value="0.3" />
   <xacro:property name="leg_radius" value="0.02" />
-  <xacro:property name="platform_x" value="0.98" />
+  <xacro:property name="platform_x" value="0.0" />
   <xacro:property name="platform_y" value="0.0" />
   <xacro:property name="platform_z" value="0.0" />
   <xacro:property name="platform_top_thickness" value="0.05"/>
+  <!-- Distances from wam_origin to platform_top_link (center of the platform) -->
+  <xacro:property name="wam_x" value="-0.22" />
+  <xacro:property name="wam_y" value="-0.14" />
+  <xacro:property name="wam_z" value="${platform_top_thickness}" />
   <xacro:property name="M_PI" value="3.1415926535897931" />
   </robot>

File: platform_description/xacro/wam_platform.urdf.xacro (robot description, xacro)
@@ -13,5 +13,5 @@
 		<parent link="platform_top_link"/>
 		<child link="wam_origin" />
-		<origin xyz="-0.22 -0.14 ${platform_top_thickness}" rpy="0.0 0.0 0.0" />
+		<origin xyz="${wam_x} ${wam_y} ${wam_z}" rpy="0.0 0.0 0.0" />
 	</joint>
 </robot>

Commit message: display.rviz axes

File: platform_description/xacro/platform.urdf.xacro (robot description, xacro)
@@ -151,5 +151,5 @@
   <joint name="imu_joint" type="fixed">
     <axis xyz="1 0 0"/> <!-- 0 1 0 -->
-    <origin rpy="0 0 0" xyz="${wam_x+0.015} ${wam_y-0.02} ${platform_top_thickness+0.0025}"/>
+    <origin rpy="0 0 0" xyz="0.0 ${wam_y-0.02} ${platform_top_thickness+0.0025}"/>
     <parent link="platform_top_link"/>
     <child link="imu_link"/>
@@ -167,5 +167,5 @@
         <gaussianNoise>0.0</gaussianNoise>
         <xyzOffset>0 0 0</xyzOffset>
-        <rpyOffset>0 0 0</rpyOffset>
+        <rpyOffset>0 0 1.0472</rpyOffset>
         <frameName>imu_link</frameName>
       </plugin>

File: platform_description/xacro/urdf/wam_platform.urdf (robot description, URDF)
Before this commit: robot wam, 19 links, 18 joints
Links:
- link imu_link: mass 0.001 -> 0.01; geometry collision box size=0.03 0.03 0.005; visual box size=0.03 0.03 0.005
- link p0_link: mass 100.0 -> 500.0
- link p1_link: mass 100.0 -> 500.0
- link platform_top_link: mass 1.0 -> 5.0
Joints:
- joint imu_joint: origin xyz=0 0 0.0 -> xyz=0.0 -0.16 0.0525 rpy=0 0 0
- joint p0_joint: limit lower=-2.0 upper=2.0 effort=1000.0 velocity=1.5 -> lower=-2.0 upper=2.0 effort=100000.0 velocity=1.5
- joint p1_joint: limit lower=-2.0 upper=2.0 effort=1000.0 velocity=1.5 -> lower=-2.0 upper=2.0 effort=100000.0 velocity=1.5
- joint world_platform_joint: origin xyz=-0.98 -0.0 -0.0 rpy=0.0 0.0 0.0 -> xyz=-0.0 -0.0 0.0 rpy=0.0 0.0 0.0

Commit message: DH convention

File: platform_description/xacro/platform.urdf.xacro (robot description, xacro)
@@ -5,5 +5,5 @@
     <inertial>
       <mass value="500.0" />
-      <origin xyz="0.0 0.0 ${platform_height/4}" />
+      <origin xyz="0 ${platform_height/4} 0" rpy="${M_PI/2} ${M_PI/2} 0" />
       <inertia ixx="3.2010" ixy="0"  ixz="0"
                iyy="3.2010" iyz="0"
@@ -11,5 +11,5 @@
     </inertial>
     <visual>
-      <origin xyz="0.0 0.0 ${platform_height/4}" rpy="0 0 0" />
+      <origin xyz="0 ${platform_height/4} 0" rpy="${M_PI/2} ${M_PI/2} 0" />
       <geometry>
         <cylinder radius="${leg_radius}" length="${platform_height/2}" />
@@ -20,5 +20,5 @@
     </visual>
     <collision>
-      <origin xyz="0.0 0.0 ${platform_height/4}" rpy="0.0 0.0 0.0" />
+        <origin xyz="0 ${platform_height/4} 0" rpy="${M_PI/2} ${M_PI/2} 0" />
       <geometry>
         <cylinder radius="${leg_radius}" length="${platform_height/2}" />
@@ -38,5 +38,5 @@
     <inertial>
       <mass value="500.0" />
-      <origin xyz="0.1 0.0 0.0" />
+      <origin xyz="0 0 0" rpy="${M_PI/2} 0 ${M_PI/2}"/>
       <inertia ixx="3.2010" ixy="0"  ixz="0"
                iyy="3.2010" iyz="0"
@@ -55,5 +55,5 @@
   <joint name="p0_joint" type="revolute" >
     <parent link="p0_link" />
-    <origin xyz="0.0 0.0 ${platform_z+platform_height/2}" rpy="0 0 0" />
+    <origin xyz="0 ${platform_z+platform_height/2} 0" rpy="${M_PI/2} 0 ${M_PI/2}" />
     <child link="p1_link" />
     <limit effort="100000.0" lower="-2.0" upper="2.0" velocity="1.5" />
@@ -75,5 +75,5 @@
     <inertial>
       <mass value="5.0" />
-      <origin xyz="0.0 0.0 ${platform_top_thickness/2}" />
+      <origin xyz="${platform_top_thickness/2} 0 0" rpy="${M_PI/2} 0 ${M_PI/2}"/>
       <inertia ixx="1.0" ixy="0"  ixz="0"
                iyy="1.0" iyz="0"
@@ -81,5 +81,5 @@
     </inertial>
     <visual>
-      <origin xyz="0.0 0.0 ${platform_top_thickness/2}" />
+        <origin xyz="${platform_top_thickness/2} 0 0" rpy="${M_PI/2} 0 ${M_PI/2}"/>
       <geometry>
         <cylinder radius="${platform_radius}" length="${platform_top_thickness}" />
@@ -90,5 +90,5 @@
     </visual>
     <collision>
-      <origin xyz="0.0 0.0 ${platform_top_thickness/2}" />
+        <origin xyz="${platform_top_thickness/2} 0 0" rpy="${M_PI/2} 0 ${M_PI/2}"/>
       <geometry>
         <cylinder radius="${platform_radius}" length="${platform_top_thickness}" />
@@ -110,5 +110,5 @@
     <child link="platform_top_link" />
     <limit effort="100000.0" lower="-2.0" upper="2.0" velocity="1.5" />
-    <axis xyz="1 0 0"/>
+    <axis xyz="0 0 1"/>
   </joint>
  <!-- p1_transmission -->

File: platform_description/xacro/properties.urdf.xacro (robot description, xacro)
@@ -9,7 +9,7 @@
   <xacro:property name="platform_top_thickness" value="0.05"/>
   <!-- Distances from wam_origin to platform_top_link (center of the platform) -->
-  <xacro:property name="wam_x" value="-0.22" />
-  <xacro:property name="wam_y" value="-0.14" />
-  <xacro:property name="wam_z" value="${platform_top_thickness}" />
+  <xacro:property name="wam_y" value="-0.22" />
+  <xacro:property name="wam_z" value="-0.14" />
+  <xacro:property name="wam_x" value="${platform_top_thickness}" />
   <xacro:property name="M_PI" value="3.1415926535897931" />
   </robot>

File: platform_description/xacro/urdf/wam_platform.urdf (robot description, URDF)
Before this commit: robot wam, 19 links, 18 joints
Joints:
- joint imu_joint: origin xyz=0.0 -0.16 0.0525 rpy=0 0 0 -> xyz=0.0 -0.24 0.0525 rpy=0 0 0
- joint p0_joint: origin xyz=0.0 0.0 0.275 rpy=0 0 0 -> xyz=0 0.275 0 rpy=1.57079632679 0 1.57079632679
- joint p1_joint: axis 1 0 0 -> 0 0 1
- joint platform_wam_joint: origin xyz=-0.22 -0.14 0.05 rpy=0.0 0.0 0.0 -> xyz=0.05 -0.22 -0.14 rpy=1.57079632679 0 1.57079632679
- joint world_platform_joint: origin xyz=-0.0 -0.0 0.0 rpy=0.0 0.0 0.0 -> xyz=-0.0 -0.0 0.0 rpy=1.57079632679 0 1.57079632679

File: platform_description/xacro/wam_platform.urdf.xacro (robot description, xacro)
@@ -7,5 +7,5 @@
 		<parent link="world"/>
 		<child link="p0_link" />
-		<origin xyz="${-platform_x} ${-platform_y} ${platform_z}" rpy="0.0 0.0 0.0" />
+		<origin xyz="${-platform_x} ${-platform_y} ${platform_z}" rpy="${M_PI/2} 0 ${M_PI/2}" />
 	</joint>
 	<xacro:include filename="$(find wam_description)/xacro/wam.urdf.xacro" />
@@ -13,5 +13,5 @@
 		<parent link="platform_top_link"/>
 		<child link="wam_origin" />
-		<origin xyz="${wam_x} ${wam_y} ${wam_z}" rpy="0.0 0.0 0.0" />
+		<origin xyz="${wam_x} ${wam_y} ${wam_z}" rpy="${M_PI/2} 0 ${M_PI/2}" />
 	</joint>
 </robot>

Commit message: imu postion fix

File: platform_description/xacro/platform.urdf.xacro (robot description, xacro)
@@ -151,5 +151,5 @@
   <joint name="imu_joint" type="fixed">
     <axis xyz="1 0 0"/> <!-- 0 1 0 -->
-    <origin rpy="0 0 0" xyz="0.0 ${wam_y-0.02} ${platform_top_thickness+0.0025}"/>
+    <origin rpy="${M_PI/2} 0 ${M_PI/2}" xyz="${platform_top_thickness+0.0025} 0 ${wam_z-0.02}"/>
     <parent link="platform_top_link"/>
     <child link="imu_link"/>

Commit message: joint position changed

File: platform_description/xacro/platform.urdf.xacro (robot description, xacro)
@@ -5,5 +5,5 @@
     <inertial>
       <mass value="500.0" />
-      <origin xyz="0 ${platform_height/4} 0" rpy="${M_PI/2} ${M_PI/2} 0" />
+      <origin xyz="0 ${p0_height/2} 0" rpy="${M_PI/2} ${M_PI/2} 0" />
       <inertia ixx="3.2010" ixy="0"  ixz="0"
                iyy="3.2010" iyz="0"
@@ -11,7 +11,7 @@
     </inertial>
     <visual>
-      <origin xyz="0 ${platform_height/4} 0" rpy="${M_PI/2} ${M_PI/2} 0" />
-      <geometry>
-        <cylinder radius="${leg_radius}" length="${platform_height/2}" />
+      <origin xyz="0 ${p0_height/2} 0" rpy="${M_PI/2} ${M_PI/2} 0" />
+      <geometry>
+        <cylinder radius="${p0_radius}" length="${p0_height}" />
       </geometry>
       <material name="Black">
@@ -20,7 +20,7 @@
     </visual>
     <collision>
-        <origin xyz="0 ${platform_height/4} 0" rpy="${M_PI/2} ${M_PI/2} 0" />
-      <geometry>
-        <cylinder radius="${leg_radius}" length="${platform_height/2}" />
+        <origin xyz="0 ${p0_height/2} 0" rpy="${M_PI/2} ${M_PI/2} 0" />
+      <geometry>
+        <cylinder radius="${p0_radius}" length="${p0_height}" />
       </geometry>
     </collision>
@@ -55,5 +55,5 @@
   <joint name="p0_joint" type="revolute" >
     <parent link="p0_link" />
-    <origin xyz="0 ${platform_z+platform_height/2} 0" rpy="${M_PI/2} 0 ${M_PI/2}" />
+    <origin xyz="0 ${platform_z+p0_height} 0" rpy="${M_PI/2} 0 ${M_PI/2}" />
     <child link="p1_link" />
     <limit effort="100000.0" lower="-2.0" upper="2.0" velocity="1.5" />
@@ -71,4 +71,45 @@
            </actuator>
   </transmission>
+  <!-- segment_top -->
+  <link name="segment_top">
+      <inertial>
+          <mass value="500.0" />
+          <origin xyz="${platform_height/2} 0 0" rpy="${M_PI/2} 0 ${M_PI/2}" />
+          <inertia ixx="3.2010" ixy="0"  ixz="0"
+                   iyy="3.2010" iyz="0"
+                   izz="0.1" />
+        </inertial>
+        <visual>
+            <origin xyz="${platform_height/2} 0 0" rpy="${M_PI/2} 0 ${M_PI/2}" />
+          <geometry>
+            <cylinder radius="${leg_radius}" length="${platform_height}" />
+          </geometry>
+          <material name="Black">
+        <color rgba="0 0 0 1.0"/>
+          </material>
+        </visual>
+        <collision>
+            <origin xyz="${platform_height/2} 0 0" rpy="${M_PI/2} 0 ${M_PI/2}" />
+          <geometry>
+            <cylinder radius="${leg_radius}" length="${platform_height}" />
+          </geometry>
+        </collision>
+  </link>
+  <gazebo reference="segment_top">
+      <material>Gazebo/Green</material>
+      <mu1>1000.0</mu1>
+      <mu2>1000.0</mu2>
+      <kp>10000000.0</kp>
+      <kd>1.0</kd>
+      <selfCollide>true</selfCollide>
+    </gazebo>
+   <!-- p1_joint -->
+   <joint name="p1_joint" type="revolute" >
+      <parent link="p1_link" />
+      <origin xyz="0.0 0.0 0.0" rpy="0 0 0" />
+      <child link="segment_top" />
+      <limit effort="100000.0" lower="-2.0" upper="2.0" velocity="1.5" />
+      <axis xyz="0 0 1"/>
+    </joint>
  <!-- platform top -->
   <link name="platform_top_link">
@@ -104,11 +145,9 @@
     <selfCollide>true</selfCollide>
   </gazebo>
- <!-- p1_joint -->
-  <joint name="p1_joint" type="revolute" >
-    <parent link="p1_link" />
-    <origin xyz="0.0 0.0 0.0" rpy="0 0 0" />
+ <!-- top_joint -->
+  <joint name="top_joint" type="fixed" >
+    <parent link="segment_top" />
+    <origin xyz="${platform_height} 0 0" rpy="0 0 0" />
     <child link="platform_top_link" />
-    <limit effort="100000.0" lower="-2.0" upper="2.0" velocity="1.5" />
-    <axis xyz="0 0 1"/>
   </joint>
  <!-- p1_transmission -->

File: platform_description/xacro/properties.urdf.xacro (robot description, xacro)
@@ -1,5 +1,5 @@
 <?xml version="1.0"?>
 <robot name="prop" xmlns:xacro="http://www.ros.org/wiki/xacro" >
-  <xacro:property name="platform_height" value="0.55" />
+  <xacro:property name="platform_height" value="0.4" />
   <xacro:property name="platform_radius" value="0.3" />
   <xacro:property name="leg_radius" value="0.02" />
@@ -7,4 +7,6 @@
   <xacro:property name="platform_y" value="0.0" />
   <xacro:property name="platform_z" value="0.0" />
+  <xacro:property name="p0_height" value="0.05" />
+  <xacro:property name="p0_radius" value="0.1" />
   <xacro:property name="platform_top_thickness" value="0.05"/>
   <!-- Distances from wam_origin to platform_top_link (center of the platform) -->
