Commit message: joint names update

File: platform_description/xacro/platform.urdf.xacro (robot description, xacro)
@@ -52,6 +52,6 @@
     <selfCollide>true</selfCollide>
   </gazebo>
- <!-- p0_joint -->
-  <joint name="p0_joint" type="revolute" >
+ <!-- platform_joint_1 -->
+  <joint name="platform_joint_1" type="revolute" >
     <parent link="p0_link" />
     <origin xyz="0 ${platform_z+p0_height} 0" rpy="${M_PI/2} 0 ${M_PI/2}" />
@@ -63,5 +63,5 @@
   <transmission name="p0_transmission">
      <type>transmission_interface/SimpleTransmission</type>
-           <joint name="p0_joint">
+           <joint name="platform_joint_1">
                 <hardwareInterface>hardware_interface/PositionJointInterface</hardwareInterface>
            </joint>
@@ -104,6 +104,6 @@
       <selfCollide>true</selfCollide>
     </gazebo>
-   <!-- p1_joint -->
-   <joint name="p1_joint" type="revolute" >
+   <!-- platform_joint_2 -->
+   <joint name="platform_joint_2" type="revolute" >
       <parent link="p1_link" />
       <origin xyz="0.0 0.0 0.0" rpy="0 0 0" />
@@ -154,5 +154,5 @@
   <transmission name="p1_transmission">
      <type>transmission_interface/SimpleTransmission</type>
-           <joint name="p1_joint">
+           <joint name="platform_joint_2">
                 <hardwareInterface>hardware_interface/PositionJointInterface</hardwareInterface>
            </joint>
@@ -190,5 +190,6 @@
   <joint name="imu_joint" type="fixed">
     <axis xyz="1 0 0"/> <!-- 0 1 0 -->
-    <origin rpy="${M_PI/2} 0 ${M_PI/2}" xyz="${platform_top_thickness+0.0025} 0 ${wam_z-0.02}"/>
+    <origin rpy="${M_PI/2} 0 ${M_PI/2}"
+    xyz="${platform_top_thickness+0.0025} ${platform_radius/2} ${platform_radius/2}"/>
     <parent link="platform_top_link"/>
     <child link="imu_link"/>
@@ -206,5 +207,5 @@
         <gaussianNoise>0.0</gaussianNoise>
         <xyzOffset>0 0 0</xyzOffset>
-        <rpyOffset>0 0 1.0472</rpyOffset>
+        <rpyOffset>0 0 1.05</rpyOffset>
         <frameName>imu_link</frameName>
       </plugin>

File: platform_description/xacro/properties.urdf.xacro (robot description, xacro)
@@ -8,5 +8,5 @@
   <xacro:property name="platform_z" value="0.0" />
   <xacro:property name="p0_height" value="0.05" />
-  <xacro:property name="p0_radius" value="0.1" />
+  <xacro:property name="p0_radius" value="0.3" />
   <xacro:property name="platform_top_thickness" value="0.05"/>
   <!-- Distances from wam_origin to platform_top_link (center of the platform) -->

File: platform_description/xacro/urdf/wam_platform.urdf (robot description, URDF)
Before this commit: robot wam, 20 links, 19 joints
Links:
- link p0_link: geometry collision cylinder length=0.05 radius=0.3; visual cylinder length=0.05 radius=0.3
Joints:
- removed joint p0_joint
- removed joint p1_joint
- added joint platform_joint_1: type revolute, parent p0_link, child p1_link, origin xyz=0 0.05 0 rpy=1.57079632679 0 1.57079632679, axis 0 1 0, limit lower=-2.0 upper=2.0 effort=100000.0 velocity=1.5
- added joint platform_joint_2: type revolute, parent p1_link, child segment_top, origin xyz=0.0 0.0 0.0 rpy=0 0 0, axis 0 0 1, limit lower=-2.0 upper=2.0 effort=100000.0 velocity=1.5
- joint imu_joint: origin xyz=0.0525 0 -0.16 rpy=1.57079632679 0 1.57079632679 -> xyz=0.0525 0.15 0.15 rpy=1.57079632679 0 1.57079632679
- joint world_platform_joint: origin xyz=-0.0 -0.0 0.0 rpy=1.57079632679 0 1.57079632679 -> xyz=-0.0 -0.0 0.0 rpy=1.57079632679 0 2.62079632679

File: platform_description/xacro/wam_platform.urdf.xacro (robot description, xacro)
@@ -7,5 +7,5 @@
 		<parent link="world"/>
 		<child link="p0_link" />
-		<origin xyz="${-platform_x} ${-platform_y} ${platform_z}" rpy="${M_PI/2} 0 ${M_PI/2}" />
+		<origin xyz="${-platform_x} ${-platform_y} ${platform_z}" rpy="${M_PI/2} 0 ${M_PI/2+1.05}" />
 	</joint>
 	<xacro:include filename="$(find wam_description)/xacro/wam.urdf.xacro" />

Commit message: tf for enu and p0_link origin fix

File: platform_description/xacro/platform.urdf.xacro (robot description, xacro)
@@ -2,8 +2,14 @@
 <robot name="platform" xmlns:xacro="http://www.ros.org/wiki/xacro" >
   <!-- P0 -->
+  <link name="platform_origin" />
+  <joint name="platform_ground" type="fixed">
+      <parent link="platform_origin"/>
+      <child link="p0_link" />
+      <origin xyz="0 ${p0_height/2} 0" rpy="0 0 0" />
+    </joint>
   <link name="p0_link">
     <inertial>
       <mass value="500.0" />
-      <origin xyz="0 ${p0_height/2} 0" rpy="${M_PI/2} ${M_PI/2} 0" />
+      <origin xyz="0 0 0" rpy="${M_PI/2} ${M_PI/2} 0" />
       <inertia ixx="3.2010" ixy="0"  ixz="0"
                iyy="3.2010" iyz="0"
@@ -11,5 +17,5 @@
     </inertial>
     <visual>
-      <origin xyz="0 ${p0_height/2} 0" rpy="${M_PI/2} ${M_PI/2} 0" />
+      <origin xyz="0 0 0" rpy="${M_PI/2} ${M_PI/2} 0" />
       <geometry>
         <cylinder radius="${p0_radius}" length="${p0_height}" />
@@ -20,5 +26,5 @@
     </visual>
     <collision>
-        <origin xyz="0 ${p0_height/2} 0" rpy="${M_PI/2} ${M_PI/2} 0" />
+        <origin xyz="0 0 0" rpy="${M_PI/2} ${M_PI/2} 0" />
       <geometry>
         <cylinder radius="${p0_radius}" length="${p0_height}" />
@@ -55,5 +61,5 @@
   <joint name="platform_joint_1" type="revolute" >
     <parent link="p0_link" />
-    <origin xyz="0 ${platform_z+p0_height} 0" rpy="${M_PI/2} 0 ${M_PI/2}" />
+    <origin xyz="0 0 0" rpy="${M_PI/2} 0 ${M_PI/2}" />
     <child link="p1_link" />
     <limit effort="100000.0" lower="-2.0" upper="2.0" velocity="1.5" />
@@ -75,5 +81,5 @@
       <inertial>
           <mass value="500.0" />
-          <origin xyz="${platform_height/2} 0 0" rpy="${M_PI/2} 0 ${M_PI/2}" />
+          <origin xyz="${platform_height/2+p0_height/2} 0 0" rpy="${M_PI/2} 0 ${M_PI/2}" />
           <inertia ixx="3.2010" ixy="0"  ixz="0"
                    iyy="3.2010" iyz="0"
@@ -81,5 +87,5 @@
         </inertial>
         <visual>
-            <origin xyz="${platform_height/2} 0 0" rpy="${M_PI/2} 0 ${M_PI/2}" />
+            <origin xyz="${platform_height/2+p0_height/2} 0 0" rpy="${M_PI/2} 0 ${M_PI/2}" />
           <geometry>
             <cylinder radius="${leg_radius}" length="${platform_height}" />
@@ -90,5 +96,5 @@
         </visual>
         <collision>
-            <origin xyz="${platform_height/2} 0 0" rpy="${M_PI/2} 0 ${M_PI/2}" />
+            <origin xyz="${platform_height/2+p0_height/2} 0 0" rpy="${M_PI/2} 0 ${M_PI/2}" />
           <geometry>
             <cylinder radius="${leg_radius}" length="${platform_height}" />

File: platform_description/xacro/urdf/wam_platform.urdf (robot description, URDF)
Before this commit: robot wam, 20 links, 19 joints
Links:
- added link platform_origin
Joints:
- added joint platform_ground: type fixed, parent platform_origin, child p0_link, origin xyz=0 0.025 0 rpy=0 0 0
- joint platform_joint_1: origin xyz=0 0.05 0 rpy=1.57079632679 0 1.57079632679 -> xyz=0 0 0 rpy=1.57079632679 0 1.57079632679
- joint world_platform_joint: child p0_link -> platform_origin

File: platform_description/xacro/wam_platform.urdf.xacro (robot description, xacro)
@@ -6,5 +6,5 @@
 	<joint name="world_platform_joint" type="fixed">
 		<parent link="world"/>
-		<child link="p0_link" />
+		<child link="platform_origin" />
 		<origin xyz="${-platform_x} ${-platform_y} ${platform_z}" rpy="${M_PI/2} 0 ${M_PI/2+1.05}" />
 	</joint>

Commit message: rviz from xacro

File: platform_description/xacro/platform.urdf.xacro (robot description, xacro)
@@ -6,10 +6,10 @@
       <parent link="platform_origin"/>
       <child link="p0_link" />
-      <origin xyz="0 ${p0_height/2} 0" rpy="0 0 0" />
+      <origin xyz="0 0 ${p0_height/2}" rpy="0 -${M_PI/2} ${M_PI}" />
     </joint>
   <link name="p0_link">
     <inertial>
       <mass value="500.0" />
-      <origin xyz="0 0 0" rpy="${M_PI/2} ${M_PI/2} 0" />
+      <origin xyz="0 0 0" rpy="0 0 0" />
       <inertia ixx="3.2010" ixy="0"  ixz="0"
                iyy="3.2010" iyz="0"
@@ -17,5 +17,5 @@
     </inertial>
     <visual>
-      <origin xyz="0 0 0" rpy="${M_PI/2} ${M_PI/2} 0" />
+      <origin xyz="0 0 0" rpy="0 ${M_PI/2} 0" />
       <geometry>
         <cylinder radius="${p0_radius}" length="${p0_height}" />
@@ -26,5 +26,5 @@
     </visual>
     <collision>
-        <origin xyz="0 0 0" rpy="${M_PI/2} ${M_PI/2} 0" />
+        <origin xyz="0 0 0" rpy="0 ${M_PI/2} 0" />
       <geometry>
         <cylinder radius="${p0_radius}" length="${p0_height}" />
@@ -44,5 +44,5 @@
     <inertial>
       <mass value="500.0" />
-      <origin xyz="0 0 0" rpy="${M_PI/2} 0 ${M_PI/2}"/>
+      <origin xyz="0 0 0" rpy="0 0 0"/>
       <inertia ixx="3.2010" ixy="0"  ixz="0"
                iyy="3.2010" iyz="0"
@@ -61,5 +61,5 @@
   <joint name="platform_joint_1" type="revolute" >
     <parent link="p0_link" />
-    <origin xyz="0 0 0" rpy="${M_PI/2} 0 ${M_PI/2}" />
+    <origin xyz="0 0 0" rpy="${M_PI/2} 0 0" />
     <child link="p1_link" />
     <limit effort="100000.0" lower="-2.0" upper="2.0" velocity="1.5" />
@@ -81,8 +81,8 @@
       <inertial>
           <mass value="500.0" />
-          <origin xyz="${platform_height/2+p0_height/2} 0 0" rpy="${M_PI/2} 0 ${M_PI/2}" />
-          <inertia ixx="3.2010" ixy="0"  ixz="0"
+          <origin xyz="${platform_height/2+p0_height/2} 0 0" rpy="0 0 0" />
+          <inertia ixx="0.1" ixy="0"  ixz="0"
                    iyy="3.2010" iyz="0"
-                   izz="0.1" />
+                   izz="3.2010" />
         </inertial>
         <visual>
@@ -122,5 +122,5 @@
     <inertial>
       <mass value="5.0" />
-      <origin xyz="${platform_top_thickness/2} 0 0" rpy="${M_PI/2} 0 ${M_PI/2}"/>
+      <origin xyz="${platform_top_thickness/2} 0 0" rpy="0 0 0"/>
       <inertia ixx="1.0" ixy="0"  ixz="0"
                iyy="1.0" iyz="0"
