Commit message: platform z and display.launch fix

File: platform_description/xacro/wam_platform.urdf.xacro (robot description, xacro)
@@ -14,5 +14,5 @@
 		<parent link="world"/>
 		<child link="p0_link" />
-		<origin xyz="${-platform_x} ${-platform_y} ${-platform_z}" rpy="0.0 0.0 0.0" />
+		<origin xyz="${-platform_x} ${-platform_y} ${platform_z}" rpy="0.0 0.0 0.0" />
 	</joint>
 	<xacro:include filename="$(find wam_description)/xacro/wam.urdf.xacro" />

Commit message: platform world joint rpy fix

File: platform_description/xacro/wam_platform.urdf.xacro (robot description, xacro)
@@ -7,5 +7,5 @@
 		<parent link="world"/>
 		<child link="platform_origin" />
-		<origin xyz="${-platform_x} ${-platform_y} ${platform_z}" rpy="${M_PI/2} 0 ${M_PI/2+1.05}" />
+		<origin xyz="${-platform_x} ${-platform_y} ${platform_z}" rpy="0 0 ${M_PI/2+1.05}" />
 	</joint>
 	<xacro:include filename="$(find wam_description)/xacro/wam.urdf.xacro" />

Commit message: world_platform_joint rpy updated

File: platform_description/xacro/wam_platform.urdf.xacro (robot description, xacro)
@@ -7,5 +7,5 @@
 		<parent link="world"/>
 		<child link="platform_origin" />
-		<origin xyz="${-platform_x} ${-platform_y} ${platform_z}" rpy="0 0 ${M_PI/2+1.05}" />
+		<origin xyz="${-platform_x} ${-platform_y} ${platform_z}" rpy="0 0 1.05" />
 	</joint>
 	<xacro:include filename="$(find wam_description)/xacro/wam.urdf.xacro" />
